Commit message: simulation env improvement

File: paws_description/urdf/paws.xacro (robot description, xacro)
@@ -276,5 +276,5 @@
     <child link="lf_link1"/>
     <axis xyz="0.0 1.0 0.0"/>
-    <dynamics damping="0.7"/>
+    <dynamics damping="0.2"/>
   </joint>
   <joint name="lf_j2" type="continuous">
@@ -283,5 +283,5 @@
     <child link="lf_link2"/>
     <axis xyz="-1.0 0.0 0.0"/>
-    <dynamics damping="0.7"/>
+    <dynamics damping="0.2"/>
   </joint>
   <joint name="lf_j3" type="continuous">
@@ -297,5 +297,5 @@
     <child link="rf_link1"/>
     <axis xyz="0.0 1.0 0.0"/>
-    <dynamics damping="0.7"/>
+    <dynamics damping="0.2"/>
   </joint>
   <joint name="rf_j2" type="continuous">
@@ -304,5 +304,5 @@
     <child link="rf_link2"/>
     <axis xyz="1.0 -0.0 -0.0"/>
-    <dynamics damping="0.7"/>
+    <dynamics damping="0.2"/>
   </joint>
   <joint name="rf_j3" type="continuous">
@@ -318,5 +318,5 @@
     <child link="lh_link1"/>
     <axis xyz="0.0 -1.0 -0.0"/>
-    <dynamics damping="0.7"/>
+    <dynamics damping="0.2"/>
   </joint>
   <joint name="lh_j2" type="continuous">
@@ -325,5 +325,5 @@
     <child link="lh_link2"/>
     <axis xyz="-1.0 -0.0 0.0"/>
-    <dynamics damping="0.7"/>
+    <dynamics damping="0.2"/>
   </joint>
   <joint name="lh_j3" type="continuous">
@@ -339,5 +339,5 @@
     <child link="rh_link1"/>
     <axis xyz="0.0 -1.0 -0.0"/>
-    <dynamics damping="0.7"/>
+    <dynamics damping="0.2"/>
   </joint>
   <joint name="rh_j2" type="continuous">
@@ -346,5 +346,5 @@
     <child link="rh_link2"/>
     <axis xyz="1.0 0.0 -0.0"/>
-    <dynamics damping="0.7"/>
+    <dynamics damping="0.2"/>
   </joint>
   <joint name="rh_j3" type="continuous">
